File: schematics/aiie.brd (EAGLE design)
At the start: 102.5 x 157.5 mm, 86 parts

Commit message: v7, mostly complete; r8, fixed USB host power
Parts:
- removed D1: 1n4001, SparkFun-DiscreteSemi:DIODE-1N4148
- removed DISPSEL: (no value), jumper:JP1
- removed LS1: SPEAKER, SparkFun-Electromechanical:PCB_MOUNT_SPEAKER
- removed MAINBAT: (no value), SparkFun-Batteries:BATTERY_18650-HOLDER
- added C2: 0.1uF, rcl:C025_050-025X075
- added C3: 47uF, Capacitor:CAPPRD508W65D1000H1100B
- added H8: MOUNT-PAD-ROUND3.0, holes:3,0-PAD
- added IC1: LM1117-TO22OH, bt_regulator:TO220L1
- added J2-PWR: (no value), SparkFun-Connectors:1X03
- added J3: SJ1-3524N, SJ1-3524N:CUI_SJ1-3524N
- added J4, J5, J6: (no value), SparkFun-Connectors:1X01
- added LS2: SPEAKER, SparkFun-Electromechanical:PCB_MOUNT_SPEAKER
- added R3, R4, R5: 3.3k, SparkFun-Resistors:AXIAL-0.3
- added R6, R7: 10k, SparkFun-Resistors:AXIAL-0.3
- added S65: (no value), SparkFun-Switches:SWITCH_SPDT_PTH_11.6X4.0MM
- added T1: 2N3904, transistor:TO92
- J1: value (none) -> ILI9341 header; device SparkFun-Connectors:1X01 -> SparkFun-Connectors:1X14
- J2: value (none) -> USB_A_PTH_MALE; device SparkFun-Connectors:1X01 -> SparkFun-Connectors:USB-A-H
- R2: value 20k -> 1k
- U$2: value SAINSMART32LCDRAW -> TEENSY41; device jorjlib:2X20 -> jorjlib:TEENSY41
- U$3: value TEENSY-3.5/3.6-BREAKOUT-REV-A2-STANDARD-NO-RAILS -> NTS2101PT1G; device Teensy-Breakout-Eagle-Library:TEENSY-3.5/3.6-BREAKOUT-REV-A2-STANDARD-NO-RAILS -> NTS2101PT1G:SOT323
- moved S64 62.6 mm to (98.3, 104.4), turned to 180 degrees
- moved R2 54.9 mm to (30.7, 132.3)
- moved R1 54.4 mm to (30.7, 142.5)
- moved J2 47.5 mm to (47.5, 139.7), turned to 270 degrees
- moved U$2 46.2 mm to (30.5, 99.1), turned to 180 degrees
- moved J1 38.7 mm to (7.62, 133.6), turned to 270 degrees
- moved CLKBAT 30.5 mm to (84.8, 124.5)
- moved U$4 21.5 mm to (79.8, 105.2), turned to 270 degrees
- moved U$3 16.0 mm to (37.6, 143.3), turned to 0 degrees
- moved H4 7.84 mm to (91.9, 92.2)
- moved C1 7.41 mm to (63.2, 138.9), turned to 180 degrees
- moved H1 7.40 mm to (8.13, 92.2)
- moved J1-PRTR 6.14 mm to (98.3, 130.6)
- moved H3 3.54 mm to (91.9, 142.2)
Connections:
- removed net DB0D15: U$2.2, U$3.15
- removed net DB10D7: U$2.17, U$3.7
- removed net DB11D8: U$2.19, U$3.8
- removed net DB12D6: U$2.21, U$3.6
- removed net DB13D20: U$2.23, U$3.20
- removed net DB14D21: U$2.25, U$3.21
- removed net DB15D5: U$2.27, U$3.5
- removed net DB1D22: U$2.4, U$3.22
- removed net DB2D23: U$2.6, U$3.23
- removed net DB3D9: U$2.8, U$3.9
- removed net DB4D10: U$2.10, U$3.10
- removed net DB5D13: U$2.12, U$3.13
- removed net DB6D11: U$2.14, U$3.11
- removed net DB7D12: U$2.16, U$3.12
- removed net DB8D2: U$2.13, U$3.2
- removed net DB9D14: U$2.15, U$3.14
- removed net LCDCS: U$2.29, U$3.18
- removed net LCDRS: U$2.7, U$3.16
- removed net LCDRST: U$2.33, U$3.19
- removed net LCDWR: U$2.9, U$3.17
- new net N$30: J2.D+, U$2.P$D+
- new net N$31: J3.2, U$2.P$D10
- new net N$32: S64.3, U$4.VCC
- new net N$33: J3.3, U$2.P$D12
- new net N$34: R3.P$1, U$4.GPIO0
- new net N$35: R4.P$1, U$4.CH_PD
- new net N$36: R5.P$1, U$4.RST
- new net N$37: U$2.P$D14, U$4.RX
- new net N$38: U$2.P$D15, U$4.TX
- new net N$39: J3.10, LS2.+
- new net N$41: R1.P$1, T1.1, U$3.1
- new net N$49: R6.P$2, U$3.3
- new net N$50: R2.P$1, U$2.P$D21
- new net N$51: C3.1, J2.VBUS, U$2.P$5V
- net GND: now also C2.1, C3.2, H8.B3,0, IC1.1, J1.2, J2-PWR.2, J2.GND, J2.SHLD1, J2.SHLD2, J3.1, J5.1, LS2.-, R7.P$1, T1.3, U$2.P$GND1, U$2.P$GND2, U$2.P$GND3, U$2.P$GND4, U$2.P$GND5, U$2.P$GND6, U$2.P$GND7; no longer DISPSEL.2, LS1.-, MAINBAT.GND@1, R2.P$1, U$2.1, U$3.AGND, U$3.GND@1, U$3.GND@2
- net N$1: now also CLKBAT.1, U$2.P$VBAT; no longer S1.1, U$3.39
- net N$10: now also S1.1, U$2.P$D38; no longer LS1.+, U$3.A21
- net N$11: now also U$2.P$D4; no longer U$3.4
- net N$12: now also J2.D-, U$2.P$D-; no longer D1.C, U$4.VCC
- net N$13: now also U$2.P$D24; no longer U$3.24
- net N$14: now also C2.2, IC1.2, J1.1, J1.8, R3.P$2, R4.P$2, R5.P$2, S64.2; no longer U$3.53, U$4.RST
- net N$15: now also U$2.P$D25; no longer U$3.25
- net N$16: now also J1.3, U$2.P$D0; no longer U$3.52, U$4.CH_PD
- net N$17: now also U$2.P$D39; no longer U$3.26
- net N$18: now also J1.4, U$2.P$D8; no longer U$3.51, U$4.TX
- net N$19: now also U$2.P$D23; no longer U$3.27
- net N$2: now also U$2.P$D33; no longer U$3.33
- net N$20: now also J1.5, U$2.P$D9; no longer U$3.40, U$4.RX
- net N$21: now also U$2.P$D28; no longer U$3.28
- net N$22: now also J1.6, U$2.P$D26; no longer U$3.41, U$4.GPIO0
- net N$23: now also U$2.P$D29; no longer U$3.29
- net N$24: now also J1.7, U$2.P$D27; no longer U$3.42, U$4.GPIO2
- net N$25: now also U$2.P$D30; no longer U$3.30
- net N$26: now also U$2.P$D31; no longer U$3.31
- net N$27: now also U$2.P$D32; no longer U$3.32
- net N$28: now also J1.9, U$2.P$D1; no longer J1.1, U$2.37
- net N$29: now also U$1.UD, U$2.P$D17; no longer DISPSEL.1, U$3.43
- net N$3: now also U$2.P$D34; no longer U$3.34
- net N$4: now also U$2.P$D35; no longer U$3.35
- net N$40: now also J2-PWR.3, J6.1, R1.P$2, U$3.2; no longer MAINBAT.PWR@1, S64.2
- net N$42: now also U$2.P$D16; no longer U$3.50
- net N$43: now also J1-PRTR.1, U$2.P$D18; no longer J1-PRTR.2, U$3.56
- net N$44: now also J1-PRTR.2, U$2.P$D19; no longer R1.P$2, R2.P$2, U$3.38
- net N$45: now also R2.P$2, T1.2; no longer J1-PRTR.1, U$3.57
- net N$46: now also J2-PWR.1, J4.1, S65.2; no longer U$1.UD, U$3.49
- net N$47: now also U$2.P$33V, U$2.P$33V2, U$2.P$33V3; no longer U$3.3V3
- net N$48: now also R6.P$1, R7.P$2, U$2.P$D20; no longer CLKBAT.1, U$3.VBAT
- net N$5: now also U$2.P$D36; no longer U$3.36
- net N$6: now also U$2.P$D37; no longer U$3.37
- net N$7: now also U$2.P$D41; no longer U$3.0
- net N$8: now also U$2.P$D3; no longer U$3.3
- net N$9: now also U$2.P$D40; no longer U$3.1
- net VCC: now also IC1.3, S65.3, U$2.P$VIN; no longer D1.A, J2.1, R1.P$1, S64.3, U$2.11, U$2.3, U$3.VIN
Routing:
- net GND: track 361.2 -> 0.00 mm, vias 1 -> 0
- net N$14: track 47.4 -> 243.6 mm
- net LCDWR: track 110.3 -> 0.00 mm
- net DB13D20: track 102.9 -> 0.00 mm, vias 3 -> 0
- net DB14D21: track 101.8 -> 0.00 mm, vias 1 -> 0
- net DB8D2: track 88.9 -> 0.00 mm, vias 8 -> 0
- net N$31: track 0.00 -> 88.6 mm
- net DB11D8: track 83.5 -> 0.00 mm, vias 4 -> 0
- net DB9D14: track 83.0 -> 0.00 mm, vias 2 -> 0
- net VCC: track 171.7 -> 91.6 mm, vias 1 -> 0
- net N$29: track 3.81 -> 79.1 mm
- net DB15D5: track 74.9 -> 0.00 mm, vias 4 -> 0
- net LCDCS: track 74.2 -> 0.00 mm, vias 3 -> 0
- net LCDRST: track 74.0 -> 0.00 mm, vias 1 -> 0
- net N$33: track 0.00 -> 71.8 mm
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- added copper zone on layer 1, net GND
- added copper zone on layer 16, net GND
Other:
- board text added: "+5"
- board text added: "+B"
- board text added: "AiiE! 20200731"
- board text added: "WiFi Power"
- board text removed: "AiiE! 20170710"
- board text removed: "Power"
