File: schematics/aiie.sch (EAGLE design)
At the start: 86 parts

Commit message: v7, mostly complete; r8, fixed USB host power
Parts:
- removed D1: 1n4001, SparkFun-DiscreteSemi:DIODE-1N4148
- removed DISPSEL: (no value), jumper:JP1E
- removed LS1: SPEAKER, SparkFun-Electromechanical:SPEAKER
- removed MAINBAT: (no value), SparkFun-Batteries:BATTERY-18650
- added C2: 0.1uF, rcl:C-EU025_050-025X075
- added C3: 47uF, Capacitor:C-POL_RADIAL-11MM-DIA
- added H8: MOUNT-PAD-ROUND3.0, holes:MOUNT-PAD-ROUND3.0
- added IC1: LM1117-TO22OH, bt_regulator:LM1117-TO22OH
- added J2-PWR: (no value), SparkFun-Connectors:CONN_03
- added J3: SJ1-3524N, SJ1-3524N:SJ1-3524N
- added J4, J5, J6: (no value), SparkFun-Connectors:CONN_01
- added LS2: SPEAKER, SparkFun-Electromechanical:SPEAKER
- added R3, R4, R5: 3.3k, SparkFun-Resistors:1KOHM-HORIZ-1/4W-1%
- added R6, R7: 10k, SparkFun-Resistors:1KOHM-HORIZ-1/4W-1%
- added S65: (no value), SparkFun-Switches:SWITCH-SPDT-PTH-11.6X4.0MM
- added T1: 2N3904, transistor:2N3904
- J1: value (none) -> ILI9341 header; device SparkFun-Connectors:CONN_01 -> SparkFun-Connectors:CONN_14
- J2: value (none) -> USB_A_PTH_MALE; device SparkFun-Connectors:CONN_01 -> SparkFun-Connectors:USB_A_PTH_MALE
- R1: device SparkFun-Resistors:10KOHM-HORIZ-1/4W-1% -> SparkFun-Resistors:1KOHM-HORIZ-1/4W-1%
- R2: value 20k -> 1k; device SparkFun-Resistors:10KOHM-HORIZ-1/4W-1% -> SparkFun-Resistors:1KOHM-HORIZ-1/4W-1%
- U$2: value SAINSMART32LCDRAW -> TEENSY41; device jorjlib:SAINSMART32LCDRAW -> jorjlib:TEENSY41
- U$3: value TEENSY-3.5/3.6-BREAKOUT-REV-A2-STANDARD-NO-RAILS -> NTS2101PT1G; device Teensy-Breakout-Eagle-Library:TEENSY-3.5/3.6-BREAKOUT-REV-A2-STANDARD-NO-RAILS -> NTS2101PT1G:NTS2101PT1G
Connections:
- removed net DB0D15: U$2.DB0, U$3.15
- removed net DB10D7: U$2.DB10, U$3.7
- removed net DB11D8: U$2.DB11, U$3.8
- removed net DB12D6: U$2.DB12, U$3.6
- removed net DB13D20: U$2.DB13, U$3.20
- removed net DB14D21: U$2.DB14, U$3.21
- removed net DB15D5: U$2.DB15, U$3.5
- removed net DB1D22: U$2.DB1, U$3.22
- removed net DB2D23: U$2.DB2, U$3.23
- removed net DB3D9: U$2.DB3, U$3.9
- removed net DB4D10: U$2.DB4, U$3.10
- removed net DB5D13: U$2.DB5, U$3.13
- removed net DB6D11: U$2.DB6, U$3.11
- removed net DB7D12: U$2.DB7, U$3.12
- removed net DB8D2: U$2.DB8, U$3.2
- removed net DB9D14: U$2.DB9, U$3.14
- removed net LCDCS: U$2.LCD_CS, U$3.18
- removed net LCDRS: U$2.LCD_RS, U$3.16
- removed net LCDRST: U$2.LCD_RST, U$3.19
- removed net LCDWR: U$2.LCD_WR, U$3.17
- new net N$30: J2.D+, U$2.P$D+
- new net N$31: J3.2, U$2.P$D10
- new net N$32: S64.S, U$4.VCC
- new net N$33: J3.3, U$2.P$D12
- new net N$34: R3.1, U$4.GPIO0
- new net N$35: R4.1, U$4.CH_PD
- new net N$36: R5.1, U$4.RST
- new net N$37: U$2.P$D14, U$4.RXD
- new net N$38: U$2.P$D15, U$4.TXD
- new net N$39: J3.10, LS2.+
- new net N$41: R1.1, T1.C, U$3.G
- new net N$49: R6.2, U$3.D
- new net N$50: R2.1, U$2.P$D21
- new net N$51: C3.+, J2.VBUS, U$2.P$5V
- net GND: now also C2.1, C3.-, H8.MOUNT, IC1.GND, J1.2, J2-PWR.2, J2.GND, J2.SHIELD, J3.1, J5.1, LS2.-, R7.1, T1.E, U$2.P$GND; no longer DISPSEL.2, LS1.-, MAINBAT.-, R2.1, U$2.GND, U$3.AGND, U$3.GND
- net N$1: now also CLKBAT.+, U$2.P$VBAT; no longer S1.1, U$3.39
- net N$10: now also S1.1, U$2.P$D38; no longer LS1.+, U$3.A21
- net N$11: now also U$2.P$D4; no longer U$3.4
- net N$12: now also J2.D-, U$2.P$D-; no longer D1.C, U$4.VCC
- net N$13: now also U$2.P$D24; no longer U$3.24
- net N$14: now also C2.2, IC1.VOUT, J1.1, J1.8, R3.2, R4.2, R5.2, S64.P; no longer U$3.53, U$4.RST
- net N$15: now also U$2.P$D25; no longer U$3.25
- net N$16: now also J1.3, U$2.P$D0; no longer U$3.52, U$4.CH_PD
- net N$17: now also U$2.P$D39; no longer U$3.26
- net N$18: now also J1.4, U$2.P$D8; no longer U$3.51, U$4.TXD
- net N$19: now also U$2.P$D23; no longer U$3.27
- net N$2: now also U$2.P$D33; no longer U$3.33
- net N$20: now also J1.5, U$2.P$D9; no longer U$3.40, U$4.RXD
- net N$21: now also U$2.P$D28; no longer U$3.28
- net N$22: now also J1.6, U$2.P$D26; no longer U$3.41, U$4.GPIO0
- net N$23: now also U$2.P$D29; no longer U$3.29
- net N$24: now also J1.7, U$2.P$D27; no longer U$3.42, U$4.GPIO2
- net N$25: now also U$2.P$D30; no longer U$3.30
- net N$26: now also U$2.P$D31; no longer U$3.31
- net N$27: now also U$2.P$D32; no longer U$3.32
- net N$28: now also J1.9, U$2.P$D1; no longer J1.1, U$2.LEDA+
- net N$29: now also U$1.UD, U$2.P$D17; no longer DISPSEL.1, U$3.43
- net N$3: now also U$2.P$D34; no longer U$3.34
- net N$4: now also U$2.P$D35; no longer U$3.35
- net N$40: now also J2-PWR.3, J6.1, R1.2, U$3.S; no longer MAINBAT.+, S64.P
- net N$42: now also U$2.P$D16; no longer U$3.50
- net N$43: now also J1-PRTR.1, U$2.P$D18; no longer J1-PRTR.2, U$3.56
- net N$44: now also J1-PRTR.2, U$2.P$D19; no longer R1.2, R2.2, U$3.38
- net N$45: now also R2.2, T1.B; no longer J1-PRTR.1, U$3.57
- net N$46: now also J2-PWR.1, J4.1, S65.P; no longer U$1.UD, U$3.49
- net N$47: now also U$2.P$33V; no longer U$3.3V3
- net N$48: now also R6.1, R7.2, U$2.P$D20; no longer CLKBAT.+, U$3.VBAT
- net N$5: now also U$2.P$D36; no longer U$3.36
- net N$6: now also U$2.P$D37; no longer U$3.37
- net N$7: now also U$2.P$D41; no longer U$3.0
- net N$8: now also U$2.P$D3; no longer U$3.3
- net N$9: now also U$2.P$D40; no longer U$3.1
- net VCC: now also IC1.VIN, S65.S, U$2.P$VIN; no longer D1.A, J2.1, R1.1, S64.S, U$2.LCD_RD, U$2.LCD_VCC, U$3.VIN
Other:
- note added: "(c) 2016-2020 Jorj Bauer <jorj@jorj.org>"
- note added: "31 Jul 2020"
- note added: "Battery voltage monitor"
- note added: "rev 8"
- note removed: "(c) 2016-2017 Jorj Bauer <jorj@jorj.org>"
- note removed: "27 Jun 2017"
- note removed: "Connect J1-J2"
- note removed: "rev 5"
- moved on the sheet: CLKBAT, H1, H3, H4, J1-PRTR, R1, R2, S1, S64, U$4
